File: core-dmx/core-dmx.kicad_pcb (KiCad board)
At the start: 2 copper layers, 44 x 54 mm, 8 parts, among them J1 XLR3, J2 XLR5, J3 Screw_Terminal_01x02, J4 Screw_Terminal_01x02, U1 MAX485E

Commit message: Various things were completed
Parts:
- added ?: , , F.Cu at (98.2, 15.8)
- moved ? 0.21 mm to (98.2, 45.1)
Other:
- board size 44 x 54 mm -> 44 x 60.7 mm
Changed lines of the file:
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@@
 	(footprint ""
 		(layer "F.Cu")
-		(at 98 45)
+		(at 98.15 15.8)
+		(property "Reference" ""
+			(at 0 0 0)
+			(layer "F.SilkS")
+			(effects
+				(font
+					(size 1.27 1.27)
+					(thickness 0.15)
+				)
+			)
+		)
+		(property "Value" ""
+			(at 0 0 0)
+			(layer "F.Fab")
+			(effects
+				(font
+					(size 1.27 1.27)
+					(thickness 0.15)
+				)
+			)
+		)
+		(property "Datasheet" ""
+			(at 0 0 0)
+			(layer "F.Fab")
+			(hide yes)
+			(effects
+				(font
+					(size 1.27 1.27)
+					(thickness 0.15)
+				)
+			)
+		)
+		(property "Description" ""
+			(at 0 0 0)
+			(layer "F.Fab")
+			(hide yes)
+			(effects
+				(font
+					(size 1.27 1.27)
+					(thickness 0.15)
+				)
+			)
+		)
+		(pad "1" thru_hole circle
+			(at 0 0)
+			(size 5.6 5.6)
+			(drill 3.2)
+			(layers "*.Cu" "*.Mask")
+			(remove_unused_layers no)
+			(zone_connect 2)
+		)
+		(embedded_fonts no)
+	)
+	(footprint ""
+		(layer "F.Cu")
+		(at 98.15 45.15)
 		(property "Reference" ""
 			(at 0 0 0)
@@
 	)
 	(gr_line
+		(start 94.7 12.3)
+		(end 101.3 12.3)
+		(stroke
+			(width 0.05)
+			(type default)
+		)
+		(layer "Edge.Cuts")
+	)
+	(gr_line
 		(start 72 19)
-		(end 114 19)
+		(end 91.05 19)
 		(stroke
 			(width 0.05)
@@
 	)
 	(gr_line
-		(start 114 19)
+		(start 114 17.25)
 		(end 114 73)
 		(stroke
 			(width 0.05)
+			(type default)
+		)
+		(layer "Edge.Cuts")
+	)
+	(gr_line
+		(start 91.05 19)
+		(end 94.7 12.3)
+		(stroke
+			(width 0.05)
+			(type default)
+		)
+		(layer "Edge.Cuts")
+	)
+	(gr_line
+		(start 103.2 17.25)
+		(end 114 17.25)
+		(stroke
+			(width 0.05)
+			(type default)
+		)
+		(layer "Edge.Cuts")
+	)
+	(gr_line
+		(start 103.2 17.25)
+		(end 101.3 12.3)
+		(stroke
+			(width 0.05)
