File: core-micro-pcb/core-micro-pcb.kicad_sch (KiCad schematic)
At the start: 0 parts

Commit message: Add core-dmx KiCad project and backup files
Added new core-dmx KiCad PCB, schematic, project, and related files, as well as backup archives. Also updated core-micro-pcb project files and added new backup and footprint cache files.
Parts:
- added J1: RJ45, symbol Connector:RJ45
- added P1: USB_C_Plug_USB2.0, symbol Connector:USB_C_Plug_USB2.0
- added U1: RP2040, Package_DFN_QFN:QFN-56-1EP_7x7mm_P0.4mm_EP3.2x3.2mm, symbol MCU_RaspberryPi:RP2040
- added U2: W5500, Package_QFP:LQFP-48_7x7mm_P0.5mm, symbol Interface_Ethernet:W5500
Connections:
- new net: P1.A1 (GND), P1.A12 (GND), P1.B1 (GND), P1.B12 (GND)
- new net: P1.A4 (VBUS), P1.A9 (VBUS), P1.B4 (VBUS), P1.B9 (VBUS)
- new net: U1.1 (IOVDD), U1.10 (IOVDD), U1.22 (IOVDD), U1.33 (IOVDD), U1.42 (IOVDD), U1.49 (IOVDD)
- new net: U1.23 (DVDD), U1.50 (DVDD)
- new net: U2.11 (AVDD), U2.15 (AVDD), U2.17 (AVDD), U2.21 (AVDD), U2.4 (AVDD), U2.8 (AVDD)
- new net: U2.14 (AGND), U2.16 (AGND), U2.19 (AGND), U2.3 (AGND), U2.48 (AGND), U2.9 (AGND)

Commit message: power pcb added
Parts:
- removed P1: USB_C_Plug_USB2.0, symbol Connector:USB_C_Plug_USB2.0
- removed U1: RP2040, Package_DFN_QFN:QFN-56-1EP_7x7mm_P0.4mm_EP3.2x3.2mm, symbol MCU_RaspberryPi:RP2040
- added C1, C10, C3, C4: 1uF, Capacitor_SMD:C_0402_1005Metric, symbol Device:C_Small
- added C11, C12, C13, C14, C15, C16, C17, C2, C7, C8: 100nF, Capacitor_SMD:C_0402_1005Metric, symbol Device:C_Small
- added C5, C6: 22pF, Capacitor_SMD:C_0402_1005Metric, symbol Device:C_Small
- added C9: 10uF, Capacitor_SMD:C_0402_1005Metric, symbol Device:C_Small
- added F1: 500mA, Fuse:Fuse_1206_3216Metric, symbol Device:Polyfuse_Small
- added J1: SWD, Connector_PinSocket_2.54mm:PinSocket_1x05_P2.54mm_Vertical, symbol Connector_Generic:Conn_01x05
- added J2: 47219-2001, 47219-2001:MOLEX_47219-2001, symbol 47219-2001:47219-2001
- added J4, J7, J8: USB_C_Receptacle_USB2.0, Connector_USB:USB_C_Receptacle_HRO_TYPE-C-31-M-12, symbol Connector:USB_C_Receptacle_USB2.0
- added J5: RJ45, symbol Connector:RJ45
- added J6: USB_A_Stacked, symbol Connector:USB_A_Stacked
- added J9: Conn_Coaxial_Small, Connector_Coaxial:U.FL_Molex_MCRF_73412-0110_Vertical, symbol Connector:Conn_Coaxial_Small
- added R1, R4, R5: 1k, Resistor_SMD:R_0402_1005Metric, symbol Device:R_Small
- added R2, R3: 27R, Resistor_SMD:R_0603_1608Metric, symbol Device:R_Small
- added R6, R7: 5k1, Resistor_SMD:R_0402_1005Metric, symbol Device:R_Small
- added SW1: SW_Push, Connector_PinSocket_2.54mm:PinSocket_1x02_P2.54mm_Vertical, symbol Switch:SW_Push
- added U1: RP2040, Sleep-Lib:RP2040-QFN-56, symbol Sleep-lib:RP2040
- added U10: PN5321A3HN_C1xx, Package_DFN_QFN:HVQFN-40-1EP_6x6mm_P0.5mm_EP4.1x4.1mm, symbol RF_NFC:PN5321A3HN_C1xx
- added U2: W25Q128JVS, Package_SO:SOIC-8_5.23x5.23mm_P1.27mm, symbol Memory_Flash:W25Q128JVS
- added U3: XC6206PxxxMR-Regulator_Linear, Package_TO_SOT_SMD:SOT-23, symbol kicad-keyboard-parts:XC6206PxxxMR-Regulator_Linear
- added U4: USBLC6-2SC6, Package_TO_SOT_SMD:SOT-23-6, symbol Power_Protection:USBLC6-2SC6
- added U5: SP706SEN-L/TR, NSOIC-8, symbol SP706SEN-L/TR:SP706SEN-L_TR
- added U6: PCF8563T/5_518, U_SO8_NXP, symbol PCF8563T/5,518:PCF8563T_5_518
- added U7: LAN9514i, Package_DFN_QFN:QFN-64-1EP_9x9mm_P0.5mm_EP7.3x7.3mm, symbol Interface_Ethernet:LAN9514i
- added U9: USB2514BI-AEZG, USB2514BI-AEZG:QFN50P600X600X100-37N, symbol USB2514BI-AEZG:USB2514BI-AEZG
- added Y1: 12MHz, Crystal:Crystal_SMD_3225-4Pin_3.2x2.5mm, symbol Device:Crystal_GND24_Small
- renumbered J1 to J3, U2 to U8
Connections:
- new net: J8.A1 (GND), J8.A12 (GND), J8.B1 (GND), J8.B12 (GND)
- new net: J8.A4 (VBUS), J8.A9 (VBUS), J8.B4 (VBUS), J8.B9 (VBUS)
- new net: U10.11 (AVSS), U10.41 (AVSS)
- new net: J4.A1 (GND), J4.A12 (GND), J4.B1 (GND), J4.B12 (GND)
- new net: J4.A4 (VBUS), J4.A9 (VBUS), J4.B4 (VBUS), J4.B9 (VBUS)
- new net: U7.10 (VDD33A), U7.49 (VDD33A), U7.5 (VDD33A), U7.51 (VDD33A), U7.54 (VDD33A), U7.57 (VDD33A), U7.64 (VDD33A)
- new net: U7.15 (VDD18CORE), U7.38 (VDD18CORE)
- new net: U7.19 (VDD33IO), U7.27 (VDD33IO), U7.33 (VDD33IO), U7.39 (VDD33IO), U7.46 (VDD33IO)
- new net +1V1: C4.1, C7.1, C8.1, U1.23 (DVDD), U1.45 (VREG_VOUT), U1.50 (DVDD)
- new net +3V3: C10.1, C11.1, C12.1, C13.1, C14.1, C15.1, C16.1, C17.1, C2.1, C3.2, C9.1, J1.2 (Pin_2), R1.1, U1.1 (IOVDD), U1.10 (IOVDD), U1.22 (IOVDD), U1.33 (IOVDD), U1.42 (IOVDD), U1.43 (ADC_AVDD), U1.44 (VREG_VIN), U1.48 (USB_VDD), U1.49 (IOVDD), U2.8 (VCC), U3.2 (VO)
- new net +5V: C1.2, F1.2, U3.3 (VI), U4.5 (VBUS)
- new net CC1: J7.A5 (CC1), R6.1
- new net CC2: J7.B5 (CC2), R7.1
- new net CS: R4.2, U1.56 (QSPI_SS_N), U2.1 (~{CS})
- new net D_+: R2.2, U1.47 (D+)
- new net D_-: R3.2, U1.46 (D-)
- new net D_N: R3.1, U4.3 (I/O2)
- new net D_P: R2.1, U4.1 (I/O1)
- new net D_USB_N: J7.A7 (D-), J7.B7 (D-), U4.4 (I/O2)
- new net D_USB_P: J7.A6 (D+), J7.B6 (D+), U4.6 (I/O1)
- new net GND: C1.1, C10.2, C11.2, C12.2, C13.2, C14.2, C15.2, C16.2, C17.2, C2.2, C3.1, C4.2, C5.1, C6.1, C7.2, C8.2, C9.2, J1.3 (Pin_3), J7.A1 (GND), J7.A12 (GND), J7.B1 (GND), J7.B12 (GND), J7.S1 (SHIELD), R6.2, R7.2, SW1.1, U1.19 (TESTEN), U1.57 (GND), U2.4 (GND), U3.1 (GND), U4.2 (GND), Y1.2, Y1.4
- new net QSPI_CLK: U1.52 (QSPI_SCLK), U2.6 (CLK)
- new net SD0: U1.53 (QSPI_SD0), U2.5 (DI(IO0))
- new net SD1: U1.55 (QSPI_SD1), U2.2 (DO(IO1))
- new net SD2: U1.54 (QSPI_SD2), U2.3 (IO2)
- new net SD3: U1.51 (QSPI_SD3), U2.7 (IO3)
- new net SWCLK: J1.5 (Pin_5), U1.24 (SWCLK)
- new net SWD: J1.4 (Pin_4), U1.25 (SWDIO)
- new net VBUS: F1.1, J7.A4 (VBUS), J7.A9 (VBUS), J7.B4 (VBUS), J7.B9 (VBUS)
- new net XTAL_IN: C5.2, U1.20 (XTAL_IN), Y1.3
- new net XTAL_O: C6.2, R5.1, Y1.1
- new net XTAL_OUT: R5.2, U1.21 (XTAL_OUT)
- new net ~{RESET}: J1.1 (Pin_1), R1.2, U1.26 (~{RUN})
- new net ~{USB_BOOT}: R4.1, SW1.2
- no-connect marks 0 -> 2
Other:
- note added: "MOUNTINGHOLES (REMOVED)"
- note added: "Maybe add something on shield?"
- moved on the sheet: J3, U8

Commit message: Various things were completed
Parts:
- removed F1: 500mA, Fuse:Fuse_1206_3216Metric, symbol Device:Polyfuse_Small
- removed J2: 47219-2001, 47219-2001:MOLEX_47219-2001, symbol 47219-2001:47219-2001
- removed J3, J5: RJ45, symbol Connector:RJ45
- removed J4, J8: USB_C_Receptacle_USB2.0, Connector_USB:USB_C_Receptacle_HRO_TYPE-C-31-M-12, symbol Connector:USB_C_Receptacle_USB2.0
- removed J6: USB_A_Stacked, symbol Connector:USB_A_Stacked
- removed J9: Conn_Coaxial_Small, Connector_Coaxial:U.FL_Molex_MCRF_73412-0110_Vertical, symbol Connector:Conn_Coaxial_Small
- removed U10: PN5321A3HN_C1xx, Package_DFN_QFN:HVQFN-40-1EP_6x6mm_P0.5mm_EP4.1x4.1mm, symbol RF_NFC:PN5321A3HN_C1xx
- removed U5: SP706SEN-L/TR, NSOIC-8, symbol SP706SEN-L/TR:SP706SEN-L_TR
- removed U6: PCF8563T/5_518, U_SO8_NXP, symbol PCF8563T/5,518:PCF8563T_5_518
- removed U7: LAN9514i, Package_DFN_QFN:QFN-64-1EP_9x9mm_P0.5mm_EP7.3x7.3mm, symbol Interface_Ethernet:LAN9514i
- removed U9: USB2514BI-AEZG, USB2514BI-AEZG:QFN50P600X600X100-37N, symbol USB2514BI-AEZG:USB2514BI-AEZG
- added C15, C16: 100nF, Capacitor_SMD:C_0402_1005Metric, symbol Device:C
- added C2, C6: 1uF, Capacitor_SMD:C_0402_1005Metric, symbol Device:C_Small
- added C20: 1nF, Capacitor_SMD:C_0402_1005Metric, symbol Device:C
- added C3: 100nF, Capacitor_SMD:C_0402_1005Metric, symbol Device:C_Small
- added C7: 1uF, Capacitor_SMD:C_0402_1005Metric, symbol Device:C
- added D1: LED, LED_SMD:LED_0201_0603Metric, symbol Device:LED
- added FB1, FB2: FerriteBead, Inductor_SMD:L_0603_1608Metric, symbol Device:FerriteBead
- added J1, J2, J3, J4, J5, J6: Screw_Terminal_01x02, TerminalBlock:TerminalBlock_Xinya_XY308-2.54-2P_1x02_P2.54mm_Horizontal, symbol Connector:Screw_Terminal_01x02
- added J9: HR911105A, HR911105A:HANRUN_HR911105A, symbol HR911105A:HR911105A
- added R1, R5: R, Resistor_SMD:R_0402_1005Metric, symbol Device:R
- added R10, R12, R9: 10k, Resistor_SMD:R_0402_1005Metric, symbol Device:R
- added R13, R14, R8: 1k, Resistor_SMD:R_0402_1005Metric, symbol Device:R
- J7: footprint Connector_USB:USB_C_Receptacle_HRO_TYPE-C-31-M-12 -> TYPE-C-31-M-12:HRO_TYPE-C-31-M-12
- U1: footprint Sleep-Lib:RP2040-QFN-56 -> Package_DFN_QFN:QFN-56-1EP_7x7mm_P0.4mm_EP3.2x3.2mm_ThermalVias
- U2: footprint Package_SO:SOIC-8_5.23x5.23mm_P1.27mm -> W25Q128JVSIM:SOIC127P790X216-8N
- renumbered C6 to C10, C7 to C11, C8 to C12, C9 to C13, C10 to C14, C11 to C17, C12 to C18, C13 to C19, C14 to C21, C15 to C22, C16 to C23, C17 to C24, C2 to C4, C3 to C5, C4 to C8, C5 to C9, J1 to J8, R4 to R11, R5 to R15, R1 to R2, R2 to R3, R3 to R4, R7 to R6, R6 to R7, U8 to U4, U4 to U5
Connections:
- net +3V3: now also U4.11 (AVDD), U4.15 (AVDD), U4.17 (AVDD), U4.21 (AVDD), U4.28 (VDD), U4.4 (AVDD), U4.8 (AVDD), C2.1, C3.1, C6.1, FB1.1, FB2.1, R1.1, R5.1
- net +5V: now also J1.2 (Pin_2)
- net GND: now also U4.14 (AGND), U4.16 (AGND), U4.19 (AGND), U4.29 (GND), U4.3 (AGND), U4.48 (AGND), U4.9 (AGND), C15.2, C16.2, C2.2, C20.2, C3.2, C6.2, C7.2, D1.1 (K), J1.1 (Pin_1), J9.10, J9.11, J9.8, R10.1, R12.1, R9.1
- net SDA: now reaches U1.11 (GPIO8)
- net SDA: now also J6.2 (Pin_2), R5.2
- net SCL: now reaches U1.12 (GPIO9)
- net SCL: now also J6.1 (Pin_1), R1.2
- net DMX1: now reaches U1.13 (GPIO10)
- net DMX1: now also J2.2 (Pin_2)
- net DMX2: now reaches U1.14 (GPIO11)
- net DMX2: now also J3.2 (Pin_2)
- net DMX3: now reaches U1.15 (GPIO12)
- net DMX3: now also J4.2 (Pin_2)
- net DMX4: now reaches U1.16 (GPIO13)
- net DMXE1: now reaches U1.17 (GPIO14)
- net DMXE1: now also J2.1 (Pin_1)
- net DMXE2: now reaches U1.18 (GPIO15)
- net DMXE2: now also J3.1 (Pin_1)
- net SURFACERX: now reaches U1.2 (GPIO0)
- net SURFACERX: now also J5.2 (Pin_2)
- net MISO: now reaches U1.27 (GPIO16)
- net MISO: now also U4.34 (MISO)
- net SCS: now reaches U1.28 (GPIO17)
- net SCS: now also U4.32 (~{SCS})
- net SCLK: now reaches U1.29 (GPIO18)
- net SCLK: now also U4.33 (SCLK)
- net SURFACETX: now reaches U1.3 (GPIO1)
- net SURFACETX: now also J5.1 (Pin_1)
- net MOSI: now reaches U1.30 (GPIO19)
- net MOSI: now also U4.35 (MOSI)
- net RST: now reaches U1.31 (GPIO20)
- net RST: now also U4.37 (~{RST})
- net INT: now reaches U1.32 (GPIO21)
- net INT: now also U4.36 (~{INT})
- net DMXE3: now reaches U1.34 (GPIO22)
- net DMXE3: now also J4.1 (Pin_1)
- net DMXE4: now reaches U1.35 (GPIO23)
- net at U1.6 (GPIO4): now also R8.2
- net TX-: now reaches U4.1 (TXN)
- net TX-: now also J9.2
- net TX+: now reaches U4.2 (TXP)
- net TX+: now also J9.1
- net at U4.22 (1V2O): now also C7.1
- net at U4.25 (LINKLED): now also R13.1
- net at U4.27 (ACTLED): now also R14.1
- net at U4.43 (PMODE2): now also R9.2
- net at U4.44 (PMODE1): now also R10.2
- net at U4.45 (PMODE0): now also R12.2
- net RX-: now reaches U4.5 (RXN)
- net RX-: now also J9.6
- net RX+: now reaches U4.6 (RXP)
- net RX+: now also J9.3
- net VBUS: no longer names the net of J7.A4 (VBUS), J7.A9 (VBUS), J7.B4 (VBUS), J7.B9 (VBUS)
- new net: D1.2 (A), R8.1
- new net: C15.1, FB1.2, J9.5
- new net: C20.1, J9.15 (SHIELD), J9.16 (SHIELD)
- new net: C16.1, FB2.2, J9.4
- new net ACTLED: J9.12, R14.2
- new net LINKLED: J9.9, R13.2
Other:
- moved on the sheet: C1, C10, C11, C12, C13, C14, C17, C18, C19, C21, C22, C23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
