File: core-micro-surface/core-micro-surface.kicad_pcb (KiCad board)
At the start: 2 copper layers, 230 x 153 mm, 151 parts, among them J1 SWD, J2 AUX ADC CONNECTION, J3 USB_B, J4 Screw_Terminal_01x04, SW1 SW_Push, SW10 SW_Push, SW11 SW_Push, SW12 SW_Push, SW13 SW_Push, SW14 SW_Push, SW15 SW_Push, SW16 SW_Push, SW17 SW_Push, SW18 SW_Push, SW19 SW_Push, SW2 SW_Push, SW20 SW_Push, SW21 SW_Push, SW22 SW_Push, SW23 SW_Push, SW24 SW_Push, SW25 SW_Push, SW26 SW_Push, SW27 SW_Push, SW28 SW_Push, SW29 SW_Push, SW3 SW_Push, SW30 SW_Push, SW31 SW_Push, SW32 SW_Push, SW33 SW_Push, SW34 SW_Push, SW35 SW_Push, SW36 SW_Push, SW37 SW_Push, SW38 SW_Push, SW39 SW_Push, SW4 SW_Push, SW40 SW_Push, SW41 SW_Push, SW42 SW_Push, SW43 SW_Push, SW44 SW_Push, SW45 SW_Push, SW46 RotaryEncoder_Switch, SW47 RotaryEncoder_Switch, SW48 RotaryEncoder_Switch, SW5 SW_Push, SW6 SW_Push, SW7 SW_Push, SW8 SW_Push, SW9 SW_Push, U1 RP2040, U2 W25Q128JVS, U3 XC6206PxxxMR-Regulator_Linear, U4 USBLC6-2SC6, U5 ADS1115IDGS, Y1 12MHz

Commit message: Various things were completed
Parts:
- added R6: 4.7k, Resistor_SMD:R_0402_1005Metric, F.Cu at (140.1, 62.5)
- added R7: 4.7k, Resistor_SMD:R_0402_1005Metric, F.Cu at (139.1, 62.5)
- J2: value AUX ADC CONNECTION -> AudioPlug2
Connections:
- RV1 pad 3: +3V3 -> +3.3V
- RV2 pad 3: +3V3 -> +3.3V
- RV3 pad 3: +3V3 -> +3.3V
- RV4 pad 3: +3V3 -> +3.3V
- RV5 pad 3: +3V3 -> +3.3V
- U5 pad 8: +3V3 -> +3.3V
Routing:
- net +3V3: track 406.3 -> 423.9 mm, vias 10 -> 11
- net SCL: track 158.0 -> 162.2 mm
- net C5: track 196.8 -> 193.4 mm
- net GND: track 738.0 -> 735.2 mm, vias 8 -> 14
- net SDA: track 164.9 -> 165.7 mm
Other:
- board text added: "CORE-MICRO-SURFACE V1"
- board text added: "ZEEROLUX"
