File: core-micro-surface/core-micro-surface.kicad_sch (KiCad schematic)
At the start: 140 parts, among them J1 SWD, J2 AudioPlug2, J3 USB_B, J4 Screw_Terminal_01x04, SW1 SW_Push, SW10 SW_Push, SW11 SW_Push, SW12 SW_Push, SW13 SW_Push, SW14 SW_Push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

Commit message: Various things were completed
Parts:
- added R6, R7: 4.7k, Resistor_SMD:R_0402_1005Metric, symbol Device:R
Connections:
- net +3.3V: now also R6.1, R7.1
- net SCL: now also R6.2
- net SDA: now also R7.2
