File: pcb/core-dmx/core-dmx.kicad_pcb (KiCad board)
At the start: 2 copper layers, 44 x 60.7 mm, 9 parts, among them J1 XLR3, J2 XLR5, J3 Screw_Terminal_01x02, J4 Screw_Terminal_01x02, U1 MAX485E

Commit message: added bom
Parts:
- J3, J4: footprint TerminalBlock_4Ucon:TerminalBlock_4Ucon_1x02_P3.50mm_Horizontal -> TerminalBlock:TerminalBlock_Xinya_XY308-2.54-2P_1x02_P2.54mm_Horizontal
